File: boards/detector/detector.kicad_pcb (KiCad board)
At the start: 2 copper layers, 110 x 115 mm, 21 parts, among them J1 CO, J2 Smoke, Q1 MMBT2222A, Q2 MMBT2222A, SW1 Button, U1 ESP32

Commit message: fixed some mistakes on pcb
Changed lines of the file:
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@@
 			(at 0 -4.2 0)
 			(layer "F.SilkS")
+			(hide yes)
 			(effects
 				(font
@@
 			(at 0 -4.2 0)
 			(layer "F.SilkS")
+			(hide yes)
 			(effects
 				(font
@@
 			(at 0 -4.2 0)
 			(layer "F.SilkS")
+			(hide yes)
 			(effects
 				(font
@@
 	)
 	(segment
-		(start 145.15304 137.58904)
-		(end 146.115 136.62708)
+		(start 103.22673 96.22673)
+		(end 104.121005 97.121005)
 		(width 1)
 		(layer "F.Cu")
@@
 	)
 	(segment
-		(start 103.4345 96.4345)
-		(end 104.121005 97.121005)
+		(start 164.893553 136.353553)
+		(end 168.026207 139.486207)
 		(width 1)
 		(layer "F.Cu")
@@
 	)
 	(segment
-		(start 123 137.5)
-		(end 123 137)
+		(start 146.54 135.787866)
+		(end 146.54 135)
 		(width 1)
 		(layer "F.Cu")
@@
 	)
 	(segment
-		(start 164.893553 136.353553)
-		(end 168.026207 139.486207)
+		(start 124.666136 138.976)
+		(end 141.804624 138.976)
 		(width 1)
 		(layer "F.Cu")
@@
 	)
 	(segment
-		(start 103.535644 54.926644)
+		(start 102.948227 55.51406)
 		(end 104.394815 54.067474)
 		(width 1)
@@
 	)
 	(segment
-		(start 102.649 57.067195)
-		(end 102.649 94.538135)
+		(start 102.649 56.236458)
+		(end 102.649 94.831967)
+		(width 1)
+		(layer "F.Cu")
+		(net 13)
+	)
+	(segment
+		(start 123 137)
+		(end 123 137.5)
 		(width 1)
 		(layer "F.Cu")
@@
 	)
 	(segment
-		(start 114 107.253963)
-		(end 114 123.746036)
+		(start 123.353553 138.353553)
+		(end 123.488 138.488)
 		(width 1)
 		(layer "F.Cu")
@@
 	)
 	(segment
-		(start 141.804624 138.976)
-		(end 124.666136 138.976)
+		(start 145.15304 137.58904)
+		(end 146.115 136.62708)
+		(width 1)
+		(layer "F.Cu")
+		(net 13)
+	)
+	(segment
+		(start 114 107.253963)
+		(end 114 123.746036)
 		(width 1)
 		(layer "F.Cu")
@@
 	)
 	(segment
+		(start 146.115 136.62708)
+		(end 146.247107 136.494973)
+		(width 1)
+		(layer "F.Cu")
+		(net 13)
+	)
+	(segment
 		(start 105.36 97.22)
 		(end 104.64 97.22)
@@
 	)
 	(segment
-		(start 123.353553 138.353553)
-		(end 123.488 138.488)
-		(width 1)
-		(layer "F.Cu")
-		(net 13)
-	)
-	(segment
-		(start 146.54 135.038855)
-		(end 146.54 135.60104)
+		(start 146.54 135.07771)
+		(end 146.54 135)
 		(width 1)
 		(layer "F.Cu")
@@
 	)
 	(segment
-		(start 147.501145 136.038855)
-		(end 146.567474 135.105184)
+		(start 147.900557 136.438267)
+		(end 146.54 135.07771)
 		(width 1)
 		(layer "F.Cu")
@@
 	)
 	(segment
-		(start 149.821554 137)
+		(start 149.2567 137)
 		(end 163.177867 137)
 		(width 1)
@@
 	)
 	(arc
-		(start 164.54 135.5)
-		(mid 164.631885 135.961939)
-		(end 164.893553 136.353553)
+		(start 123 137.5)
+		(mid 123.091885 137.961939)
+		(end 123.353553 138.353553)
 		(width 1)
 		(layer "F.Cu")
@@
 	(arc
 		(start 164.54 135.5)
-		(mid 164.54 135.5)
-		(end 164.54 135.5)
+		(mid 164.631885 135.961939)
+		(end 164.893553 136.353553)
 		(width 1)
 		(layer "F.Cu")
@@
 	)
 	(arc
-		(start 123.488 138.488)
-		(mid 124.028533 138.849172)
-		(end 124.666136 138.976)
+		(start 164.54 135.5)
+		(mid 164.54 135.5)
+		(end 164.54 135.5)
 		(width 1)
 		(layer "F.Cu")
@@
 	)
 	(arc
-		(start 106.828111 97.828111)
-		(mid 106.154536 97.378042)
-		(end 105.36 97.22)
+		(start 123.488 138.488)
+		(mid 124.028533 138.849172)
+		(end 124.666136 138.976)
 		(width 1)
 		(layer "F.Cu")
@@
 	)
 	(arc
-		(start 102.649 94.538135)
-		(mid 102.853144 95.56444)
-		(end 103.4345 96.4345)
+		(start 106.828111 97.828111)
+		(mid 106.154536 97.378042)
+		(end 105.36 97.22)
 		(width 1)
 		(layer "F.Cu")
@@
 	)
 	(arc
-		(start 147.501145 136.038855)
-		(mid 148.565757 136.750206)
-		(end 149.821554 137)
+		(start 102.649 94.831967)
+		(mid 102.799147 95.586807)
+		(end 103.22673 96.22673)
 		(width 1)
 		(layer "F.Cu")
@@
 	)
 	(arc
-		(start 146.54 135.038855)
-		(mid 146.54714 135.074752)
-		(end 146.567474 135.105184)
+		(start 147.900557 136.438267)
+		(mid 148.522761 136.85401)
+		(end 149.2567 137)
 		(width 1)
 		(layer "F.Cu")
@@
 	)
 	(arc
-		(start 146.54 135.60104)
-		(mid 146.429546 136.156329)
-		(end 146.115 136.62708)
+		(start 141.804624 138.976)
+		(mid 143.616773 138.61554)
+		(end 145.15304 137.58904)
 		(width 1)
 		(layer "F.Cu")
@@
 	)
 	(arc
-		(start 123 137.5)
-		(mid 123.091885 137.961939)
-		(end 123.353553 138.353553)
+		(start 146.54 135.787866)
+		(mid 146.46388 136.170549)
+		(end 146.247107 136.494973)
 		(width 1)
 		(layer "F.Cu")
@@
 	)
 	(arc
-		(start 103.535644 54.926644)
-		(mid 102.879431 55.908737)
-		(end 102.649 57.067195)
-		(width 1)
-		(layer "F.Cu")
-		(net 13)
-	)
-	(arc
-		(start 145.15304 137.58904)
-		(mid 143.616773 138.61554)
-		(end 141.804624 138.976)
+		(start 102.948227 55.51406)
+		(mid 102.726766 55.845499)
+		(end 102.649 56.236458)
 		(width 1)
 		(layer "F.Cu")
@@
 			)
 		)
-	)
-	(zone
-		(net 13)
-		(net_name "VCC")
-		(layer "F.Cu")
-		(hatch edge 0.5)
-		(priority 3)
-		(connect_pads
-			(clearance 0.5)
-		)
-		(min_thickness 0.25)
-		(filled_areas_thickness no)
-		(fill yes
-			(thermal_gap 0.5)
-			(thermal_bridge_width 1)
-		)
-		(polygon
-			(pts
-				(xy 146.75 135.75) (xy 145 138.25) (xy 148.25 137) (xy 148.25 136.25)
-			)
-		)
